File: CAD Examples/Basic_example/Basic_example.kicad_sch (KiCad schematic)
At the start: 2 parts, among them U2 ELPM-S3LW

Commit message: update design
Parts:
- added 3V3, DTR, GND, RST, RXD, TXD: TestPoint, symbol Connector:TestPoint
- added C2: 22uF, Capacitor_SMD:C_0402_1005Metric, symbol Device:C
- added C3, C4: 12pF, Capacitor_SMD:C_0402_1005Metric, symbol Device:C
- added C5: 10uF, Capacitor_SMD:C_0402_1005Metric, symbol Device:C
- added R1: 10K, Resistor_SMD:R_0402_1005Metric, symbol Device:R
- added SW1: Reset, Button_Switch_SMD:SW_Push_SPST_NO_Alps_SKRK, symbol Switch:SW_Push
- added Y1: 32.768KHz, Crystal:Crystal_SMD_2012-2Pin_2.0x1.2mm, symbol Device:Crystal
- C1: value 100nF -> 1uF
- renumbered U2 to U1
Connections:
- net GND: now also C2.2, C3.2, C4.2, C5.2, GND.1, SW1.1
- net +3V3: now reaches C1.1, U1.11 (3V3_ESP)
- net +3V3: now also U1.27 (3V3_LORA), U1.28 (VDD_RTC), U1.30 (PWR_LED), 3V3.1, C2.1, R1.1
- net SDA: now reaches U1.14 (GPIO8/SDA)
- net SCL: now reaches U1.15 (GPIO9/SCL)
- net GPIO15: now reaches U1.16 (GPIO15/XTAL_P)
- net GPIO16: now reaches U1.17 (GPIO16/XTAL_N)
- net ~{RESET}: now reaches U1.2 (RESET)
- net ~{RESET}: now also C5.1, R1.2, RST.1, SW1.2
- net DTR: now reaches U1.3 (GPIO0)
- net DTR: now also DTR.1
- net RXD: now reaches U1.55 (RXD)
- net RXD: now also RXD.1
- net TXD: now reaches U1.56 (TXD)
- net TXD: now also TXD.1
- new net GPIO_15: C3.1, Y1.1
- new net GPIO_16: C4.1, Y1.2
- no-connect marks 0 -> 12
Other:
- note added: "DEEP STOP I/O"
- note added: "ELPM-S3LW: Basic example"
- note added: "Prog test points"
- note added: "RESERVED LORA"
- company: (none) -> OBJEX
- title: (none) -> Basic example
- moved on the sheet: C1, U1
